File: ECAD/Localisation-2025/Localisation-2025.kicad_sch (KiCad schematic)
At the start: 17 parts, among them J1 Serial_Strategy, J2 Serial_Lidar, J4 Oled, U2 AMS1117-3.3, U3 Teensy4.0

Commit message: save minor changes
Parts:
- J4: value Oled -> BNO0xx
- R2, R3: value R_Small -> 10k
Changed lines of the file:
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@@
 	(wire
 		(pts
+			(xy 116.84 38.1) (xy 118.11 38.1)
+		)
+		(stroke
+			(width 0)
+			(type default)
+		)
+	)
+	(wire
+		(pts
 			(xy 175.26 73.66) (xy 179.07 73.66)
 		)
@@
 		)
 	)
+	(text_box "Si BNO085, pas de R_pullup"
+		(exclude_from_sim no)
+		(at 111.76 16.51 0)
+		(size 15.24 7.62)
+		(stroke
+			(width 0)
+			(type default)
+		)
+		(fill
+			(type none)
+		)
+		(effects
+			(font
+				(size 1.27 1.27)
+			)
+			(justify left top)
+		)
+	)
 	(global_label "RX"
 		(shape input)
@@
 			)
 		)
-		(property "Value" "R_Small"
+		(property "Value" "10k"
 			(at 99.06 27.9399 0)
 			(effects
@@
 			)
 		)
-		(property "Value" "R_Small"
+		(property "Value" "10k"
 			(at 107.95 27.9399 0)
 			(effects
@@
 	(symbol
 		(lib_id "power:+3.3V")
-		(at 118.11 38.1 90)
+		(at 116.84 38.1 90)
 		(unit 1)
 		(exclude_from_sim no)
@@
 		(fields_autoplaced yes)
 		(property "Reference" "#PWR0121"
-			(at 121.92 38.1 0)
+			(at 120.65 38.1 0)
 			(effects
 				(font
@@
 		)
 		(property "Value" "+3V3"
-			(at 119.38 38.0999 90)
+			(at 113.03 38.0999 90)
 			(effects
 				(font
 					(size 1.27 1.27)
 				)
-				(justify right)
+				(justify left)
 			)
 		)
 		(property "Footprint" ""
-			(at 118.11 38.1 0)
+			(at 116.84 38.1 0)
 			(effects
 				(font
@@
 		)
 		(property "Datasheet" ""
-			(at 118.11 38.1 0)
+			(at 116.84 38.1 0)
 			(effects
 				(font
@@
 		)
 		(property "Description" ""
-			(at 118.11 38.1 0)
+			(at 116.84 38.1 0)
 			(effects
 				(font
@@
 			)
 		)
-		(property "Value" "Oled"
+		(property "Value" "BNO0xx"
 			(at 116.84 31.75 0)
 			(effects
