File: ECAD/PumpBoard-2025/PumpBoard-2025.kicad_pcb (KiCad board)
At the start: 2 copper layers, 62.9 x 25.4 mm, 25 parts, among them J1 Conn_01x04, J2 Conn_01x01, J3 CON_EV, J4 CON_PUMP, Q1 AO3400A, Q2 AO3400A, U1 ATtiny412-SS

Commit message: New pcb pump board
Parts:
- removed C1: C_Small, Capacitor_SMD:C_1206_3216Metric_Pad1.33x1.80mm_HandSolder
- removed J2: Conn_01x01, Connector_PinHeader_2.54mm:PinHeader_1x01_P2.54mm_Vertical
- removed R2: 470R, Resistor_SMD:R_1206_3216Metric_Pad1.30x1.75mm_HandSolder
- removed U1: ATtiny412-SS, Package_SO:SOIC-8_3.9x4.9mm_P1.27mm
- added C2: C_Polarized_Small, Capacitor_THT:CP_Radial_D10.0mm_P5.00mm, B.Cu at (147.6, 99.0)
- added G***: LOGO, LOGO, F.Cu at (134.2, 87.0)
- added G***: LOGO, LOGO, F.Cu at (156.3, 103.9)
- added kibuzzard-67A8F398: G***, kibuzzard-67A8F398, F.Cu at (151.1, 103.6)
- added kibuzzard-67A8F3A7: G***, kibuzzard-67A8F3A7, F.Cu at (148.6, 104.3)
- moved D1 2.54 mm to (153.7, 87.0)
- moved D3 2.54 mm to (156.2, 87.0)
- moved R1 2.54 mm to (153.7, 92.1)
- moved R4 2.54 mm to (156.2, 92.1)
- moved J3 0.16 mm to (137.0, 96.5)
- moved R6 0.14 mm to (158.6, 92.1)
Connections:
- J1 pad 3: signal -> S_PUMP
- J1 pad 4: TX -> S_EV
Routing:
- net TX: track 21.4 -> 0.00 mm
- net S_EV: track 5.50 -> 18.0 mm
- net S_PUMP: track 10.9 -> 17.7 mm
- net Net-(R2-Pad1): track 6.60 -> 0.00 mm
- net signal: track 5.15 -> 0.00 mm
- net Net-(J2-Pad1): track 4.06 -> 0.00 mm
- net +5V: track 82.8 -> 83.4 mm, vias 2 -> 0
- net GND: vias 6 -> 0
Other:
- board text added: "Les Karibous 2025 - Barba"
- board text added: "Produced by Aisler"
- board text removed: "G"
- board text removed: "Les Karibous 2021 - Barba"
- board text removed: "S"
