File: ECAD/PumpBoard-2025/PumpBoard-2025.kicad_sch (KiCad schematic)
At the start: 25 parts, among them J1 Conn_01x04, J2 Conn_01x01, J3 CON_EV, J4 CON_PUMP, Q1 AO3400A, Q2 AO3400A, U1 ATtiny412-SS

Commit message: New pcb pump board
Parts:
- removed C1: C_Small, Capacitor_SMD:C_1206_3216Metric_Pad1.33x1.80mm_HandSolder, symbol Device:C_Small
- removed J2: Conn_01x01, Connector_PinHeader_2.54mm:PinHeader_1x01_P2.54mm_Vertical, symbol Connector_Generic:Conn_01x01
- removed R2: 470R, Resistor_SMD:R_1206_3216Metric_Pad1.30x1.75mm_HandSolder, symbol Device:R_Small
- removed U1: ATtiny412-SS, Package_SO:SOIC-8_3.9x4.9mm_P1.27mm, symbol MCU_Microchip_ATtiny:ATtiny412-SS
- added C2: C_Polarized_Small, Capacitor_THT:CP_Radial_D10.0mm_P5.00mm, symbol Device:C_Polarized_Small
Connections:
- net TX is gone; now on net S_EV: J1.4 (Pin_4)
- net signal is gone; now on net S_PUMP: J1.3 (Pin_3)
- net +5V: now also C2.1
- net GND: now also C2.2
Other:
- moved on the sheet: D1, H1, H2, H3, H4, R1
